File: BPS6001_Classic_Computing_Shield_1.sch (KiCad schematic (older format))
At the start: 26 parts

Commit message: Revision 2, needs extra check.
Parts:
- removed CFG1: JP5Q, BPS6001 Classic Computing Shield:JP5Q, symbol BPS6001_Classic_Computing_Shield-eagle-import:JP5Q
- removed R11, R18: 47K, BPS6001 Classic Computing Shield:0603, symbol BPS6001_Classic_Computing_Shield-eagle-import:R0603
- removed S2, S5: EVQQ2, BPS6001 Classic Computing Shield:EVQ-Q2, symbol BPS6001_Classic_Computing_Shield-eagle-import:EVQQ2
- added J1: Conn_02x03_Row_Letter_Last, Connector_PinSocket_2.54mm:PinSocket_2x03_P2.54mm_Vertical, symbol Connector_Generic:Conn_02x03_Odd_Even
Connections:
- net labels added: D20, IEC-L-SRQ, SW_FUNCTION, SW_RESET, SW_SELECT, X1, X2, X3, d21
- net labels removed: RESET, SW_RIGHT
- wire segments 118 -> 98
