File: Joysticks.sch (KiCad schematic (older format))
At the start: 18 parts

Commit message: Revision 2, needs extra check.
Connections:
- wire segments 88 -> 86
Changed lines of the file:
@@
 $Descr User 16774 9150
 encoding utf-8
-Sheet 1 8
+Sheet 4 8
 Title ""
 Date ""
@@
 	7800 3000 7900 3000
 Wire Wire Line
-	7900 3000 7950 3000
-Wire Wire Line
-	7950 3000 8000 3000
-Wire Wire Line
 	8000 3000 8100 3000
 Wire Wire Line
@@
 Wire Wire Line
 	8200 3000 8300 3000
-Connection ~ 7600 3000
 Connection ~ 7700 3000
 Connection ~ 7800 3000
 Connection ~ 7900 3000
-Connection ~ 7950 3000
 Connection ~ 8000 3000
 Connection ~ 8100 3000
 Connection ~ 8200 3000
-Connection ~ 8300 3000
 Text GLabel 7600 3000 0    10   BiDi ~ 0
 JOY_3V3
@@
 	7800 1000 7900 1000
 Wire Wire Line
-	7900 1000 7950 1000
-Wire Wire Line
-	7950 1000 8000 1000
-Wire Wire Line
 	8000 1000 8100 1000
 Wire Wire Line
@@
 Wire Wire Line
 	8200 1000 8300 1000
-Connection ~ 7600 1000
 Connection ~ 7700 1000
 Connection ~ 7800 1000
 Connection ~ 7900 1000
-Connection ~ 7950 1000
 Connection ~ 8000 1000
 Connection ~ 8100 1000
 Connection ~ 8200 1000
-Connection ~ 8300 1000
 Text GLabel 7600 1000 0    10   BiDi ~ 0
 3V3_PWR6
@@
 Text Notes 12350 7250 0    59   ~ 0
 See more details at www.GadgetFactory.net
+Wire Wire Line
+	7900 3000 8000 3000
+Wire Wire Line
+	7900 1000 8000 1000
 $EndSCHEMATC
