File: RS232_IEC.sch (KiCad schematic (older format))
At the start: 13 parts, among them X2 MAB6H

Commit message: Revision 2, needs extra check.
Parts:
- removed B1: SPARKFUN_LOGIC_LEVEL_CONVERTER, BPS6001 Classic Computing Shield:SPARKFUN_LOGIC_LEVEL_CONVERTER, symbol BPS6001_Classic_Computing_Shield-eagle-import:SPARKFUN_LOGIC_LEVEL_CONVERTER
- removed C2, C4, C5, C6: 10p, BPS6001 Classic Computing Shield:C0603, symbol BPS6001_Classic_Computing_Shield-eagle-import:C-EUC0603
- removed R22, R28, R49, R50, R51: 1k, BPS6001 Classic Computing Shield:R0603, symbol BPS6001_Classic_Computing_Shield-eagle-import:R-EU_R0603
- added C40, C41, C42, C43, C44: 15pF, Capacitor_SMD:C_0603_1608Metric, symbol Device:C_Small
- added Q0, Q1, Q2, Q3, Q4: BSS138, Package_TO_SOT_SMD:SOT-323_SC-70, symbol Transistor_FET:BSS138
- added R60, R61, R62, R63, R64, R65, R66, R67, R68, R69: 10K, Resistor_SMD:R_0603_1608Metric, symbol Device:R_Small_US
- C1, C3: value 10p -> 100nF
Connections:
- net GND: no longer C3.1
- net IEC-L-ATN: now also Q3.2 (S), R66.2
- net IEC-L-CLK: now also Q2.2 (S), R64.2
- net IEC-L-DATA: now also Q1.2 (S), R62.2
- net IEC-L-RESET: now also Q0.2 (S), R60.2
- net IEC-H-DATA: now reaches X2.5
- net IEC-H-DATA: now also C41.1, Q1.3 (D), R63.2
- net IEC-H-RESET: now reaches X2.6
- net IEC-H-RESET: now also C40.1, Q0.3 (D), R61.2
- net IEC-H-ATN: now reaches X2.3
- net IEC-H-ATN: now also C43.1, Q3.3 (D), R67.2
- net IEC-H-CLK: now reaches X2.4
- net IEC-H-CLK: now also C42.1, Q2.3 (D), R65.2
- net IEC-H-SRQ: now reaches X2.1
- net IEC-H-SRQ: now also C44.1, Q4.3 (D), R69.2
- new net: Q0.1 (G), R60.1
- new net: Q1.1 (G), R62.1
- new net: Q2.1 (G), R64.1
- new net: Q3.1 (G), R66.1
- new net: Q4.1 (G), R68.1
- new net IEC-L-SRQ: Q4.2 (S), R68.2
Other:
- moved on the sheet: C1, C3, X2
