File: SD_Card.sch (KiCad schematic (older format))
At the start: 4 parts

Commit message: Revision 2, needs extra check.
Changed lines of the file:
@@
 $Descr User 16774 8268
 encoding utf-8
-Sheet 1 8
+Sheet 3 8
 Title ""
 Date ""
@@
 Text GLabel 7800 2100 2    70   BiDi ~ 0
 SD_MISO
-Connection ~ 7000 2100
 Wire Wire Line
 	8300 2200 7300 2200
