File: BPS6001 Classic Computing Shield.kicad_pcb (KiCad board)
At the start: 2 copper layers, 119.4 x 58.7 mm, 84 parts, among them X1 VGA, X2 MAB6H

Commit message: Revision 2, needs extra check.
Parts:
- removed B1: SPARKFUN_LOGIC_LEVEL_CONVERTER, BPS6001 Classic Computing Shield:SPARKFUN_LOGIC_LEVEL_CONVERTER
- removed C2, C4, C5, C6: 10p, BPS6001 Classic Computing Shield:C0603
- removed CFG1: JP5Q, BPS6001 Classic Computing Shield:JP5Q
- removed R11, R18: 47K, BPS6001 Classic Computing Shield:0603
- removed R22, R28, R49, R50, R51: 1k, BPS6001 Classic Computing Shield:R0603
- removed the S2 at (127.9, 120.8)
- removed the S3 at (157.3, 112.9)
- removed S5: EVQQ2, BPS6001 Classic Computing Shield:EVQ-Q2
- removed U$1, U$2, U$3: , BPS6001 Classic Computing Shield:STAND-OFF-TIGHT
- added C40: 15pF, Capacitor_SMD:C_0603_1608Metric, F.Cu at (175.9, 90.8)
- added C41: 15pF, Capacitor_SMD:C_0603_1608Metric, F.Cu at (189.9, 98.4)
- added C42: 15pF, Capacitor_SMD:C_0603_1608Metric, F.Cu at (189.2, 94.0)
- added C43: 15pF, Capacitor_SMD:C_0603_1608Metric, F.Cu at (189.2, 83.8)
- added C44: 15pF, Capacitor_SMD:C_0603_1608Metric, F.Cu at (189.2, 80.0)
- added J1: Conn_02x03_Row_Letter_Last, Connector_PinSocket_2.54mm:PinSocket_2x03_P2.54mm_Vertical, F.Cu at (149.9, 105.4)
- added Q0: BSS138, Package_TO_SOT_SMD:SOT-323_SC-70, F.Cu at (172.7, 90.2)
- added Q1: BSS138, Package_TO_SOT_SMD:SOT-323_SC-70, F.Cu at (189.9, 102.9)
- added Q2: BSS138, Package_TO_SOT_SMD:SOT-323_SC-70, F.Cu at (181.6, 94.0)
- added Q3: BSS138, Package_TO_SOT_SMD:SOT-323_SC-70, F.Cu at (181.6, 85.1)
- added Q4: BSS138, Package_TO_SOT_SMD:SOT-323_SC-70, F.Cu at (181.6, 80.0)
- added R60: 10K, Resistor_SMD:R_0603_1608Metric, F.Cu at (172.7, 92.7)
- added R61: 10K, Resistor_SMD:R_0603_1608Metric, F.Cu at (172.7, 87.6)
- added R62: 10K, Resistor_SMD:R_0603_1608Metric, F.Cu at (186.1, 104.8)
- added R63: 10K, Resistor_SMD:R_0603_1608Metric, F.Cu at (186.1, 101.0)
- added R64: 10K, Resistor_SMD:R_0603_1608Metric, F.Cu at (180.3, 97.2)
- added R65: 10K, Resistor_SMD:R_0603_1608Metric, F.Cu at (186.7, 94.0)
- added R66: 10K, Resistor_SMD:R_0603_1608Metric, F.Cu at (180.3, 87.6)
- added R67: 10K, Resistor_SMD:R_0603_1608Metric, F.Cu at (186.7, 83.8)
- added R68: 10K, Resistor_SMD:R_0603_1608Metric, F.Cu at (180.3, 82.5)
- added R69: 10K, Resistor_SMD:R_0603_1608Metric, F.Cu at (186.7, 80.0)
- added S1: EVQQ2, BPS6001 Classic Computing Shield:EVQ-Q2, F.Cu at (165.1, 112.4)
- C1, C3: value 10p -> 100nF
- moved R8 20.2 mm to (139.7, 124.8)
- moved R17 17.7 mm to (128.3, 112.4), turned to 270 degrees
- moved R2 14.1 mm to (162.6, 124.8)
- moved R4 14.1 mm to (157.5, 124.8)
- moved R5 14.1 mm to (154.9, 124.8)
- moved R6 14.1 mm to (152.4, 124.8)
- moved R3 14.1 mm to (160.0, 124.8)
- moved R1 12.7 mm to (166.5, 124.8)
- moved R7 12.7 mm to (149.7, 124.8)
- moved S3 11.1 mm to (137.8, 112.4)
- moved C1 10.8 mm to (187.3, 89.5), turned to 0 degrees
- moved R10 10.7 mm to (144.8, 109.2)
- moved R9 10.1 mm to (158.8, 107.3), turned to 270 degrees
- moved C3 7.89 mm to (181.6, 90.8), turned to 180 degrees
- moved S2 7.89 mm to (151.1, 112.4), turned to 180 degrees
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- renumbered S1 to S2, S4 to S3
Connections:
- AJ2 pad LS: Net-(AJ2-PadLS) -> (no net)
- AJ2 pad RS: Net-(AJ2-PadRS) -> (no net)
- H1 pad D10: JS1_7 -> SD_SCK
- H1 pad D11: JS1_2 -> SD_MOSI
- H1 pad D12: JS1_6 -> SD_MISO
- H1 pad D13: JS1_1 -> (no net)
- H1 pad D14: SD_MOSI -> JS1_5
- H1 pad D15: SD_SCK -> IEC-L-DATA
- H1 pad D16: SD_~CS -> IEC-L-CLK
- H1 pad D17: /BPS6001 Classic Computing Shield_1/SW_LEFT -> IEC-L-ATN
- H1 pad D18: /BPS6001 Classic Computing Shield_1/SW_UP -> IEC-L-RESET
- H1 pad D19: /BPS6001 Classic Computing Shield_1/RESET -> IEC-L-SRQ
- H1 pad D2: SD_MISO -> JS1_9
- H1 pad D20: /BPS6001 Classic Computing Shield_1/SW_DOWN -> (no net)
- H1 pad D21: /BPS6001 Classic Computing Shield_1/SW_RIGHT -> (no net)
- H1 pad D28: IEC-L-ATN -> SW_SELECT
- H1 pad D3: SD_CD -> JS1_4
- H1 pad D30: IEC-L-RESET -> SW_RESET
- H1 pad D4: IEC-L-CLK -> JS1_3
- H1 pad D5: IEC-L-DATA -> JS1_7
- H1 pad D6: JS1_5 -> JS1_2
- H1 pad D7: JS1_9 -> JS1_6
- H1 pad D8: JS1_4 -> JS1_1
- H1 pad D9: JS1_3 -> SD_~CS
- H1 pad RES: Net-(H1-PadRES) -> (no net)
- H1 pad RX: /BPS6001 Classic Computing Shield_1/RX -> (no net)
- H1 pad TX: /BPS6001 Classic Computing Shield_1/TX -> (no net)
- H1 pad VIN: Net-(H1-PadVIN) -> (no net)
- PS2_B1 pad 2: Net-(PS2_B1-Pad2) -> (no net)
- PS2_B1 pad 6: Net-(PS2_B1-Pad6) -> (no net)
- PWR_1 pad P2: Net-(PWR_1-PadP2) -> (no net)
- PWR_1 pad P4: Net-(PWR_1-PadP4) -> (no net)
- PWR_2 pad P2: Net-(PWR_2-PadP2) -> (no net)
- R10 pad 2: /BPS6001 Classic Computing Shield_1/SW_UP -> SW_SELECT
- R17 pad 2: /BPS6001 Classic Computing Shield_1/SW_DOWN -> SW_RESET
- R9 pad 2: /BPS6001 Classic Computing Shield_1/SW_LEFT -> SW_FUNCTION
- S2 pad A: /BPS6001 Classic Computing Shield_1/SW_UP -> SW_SELECT
- S2 pad A': /BPS6001 Classic Computing Shield_1/SW_UP -> SW_SELECT
- S3 pad A: /BPS6001 Classic Computing Shield_1/SW_DOWN -> SW_RESET
- S3 pad A': /BPS6001 Classic Computing Shield_1/SW_DOWN -> SW_RESET
- SD1 pad 1: Net-(SD1-Pad1) -> (no net)
- SD1 pad 8: Net-(SD1-Pad8) -> (no net)
- SD1 pad CD1: SD_CD -> (no net)
- SD1 pad CD2: Net-(SD1-PadCD2) -> (no net)
- X1 pad 12: Net-(X1-Pad12) -> (no net)
- X1 pad 15: Net-(X1-Pad15) -> (no net)
- X1 pad 4: Net-(X1-Pad4) -> (no net)
- X1 pad 5: Net-(X1-Pad5) -> (no net)
- X1 pad 9: Net-(X1-Pad9) -> (no net)
- X2 pad 1: Net-(R22-Pad1) -> IEC-H-SRQ
- X2 pad 3: Net-(B1-PadHV1) -> IEC-H-ATN
- X2 pad 4: Net-(B1-PadHV2) -> IEC-H-CLK
- X2 pad 5: Net-(B1-PadHV3) -> IEC-H-DATA
- X2 pad 6: Net-(B1-PadHV4) -> IEC-H-RESET
Routing:
- net IEC-L-SRQ: track 0.00 -> 74.6 mm, vias 0 -> 1
- net /BPS6001 Classic Computing Shield_1/SW_DOWN: track 67.9 -> 0.00 mm, vias 2 -> 0
- net /BPS6001 Classic Computing Shield_1/SW_RIGHT: track 66.3 -> 0.00 mm
- net /BPS6001 Classic Computing Shield_1/SW_LEFT: track 57.4 -> 0.00 mm
- net /BPS6001 Classic Computing Shield_1/SW_UP: track 56.7 -> 0.00 mm
- net /BPS6001 Classic Computing Shield_1/RESET: track 55.0 -> 0.00 mm, vias 1 -> 0
- net SW_SELECT: track 0.00 -> 52.3 mm, vias 0 -> 1
- net SD_CD: track 40.2 -> 0.00 mm, vias 1 -> 0
- net Net-(B1-PadHV3): track 36.6 -> 0.00 mm, vias 2 -> 0
- net SW_RESET: track 0.00 -> 35.6 mm, vias 0 -> 1
- net IEC-L-RESET: track 92.3 -> 59.8 mm
- net Net-(B1-PadHV1): track 31.4 -> 0.00 mm
- net IEC-L-DATA: track 33.5 -> 63.7 mm, vias 0 -> 1
- net Net-(B1-PadHV2): track 26.3 -> 0.00 mm
- net Net-(B1-PadHV4): track 22.7 -> 0.00 mm
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Other:
- board text added: "(C) deFEEST WTF"
- board text added: "C64 Shield V1.337"
- board text added: "Copyright Paul Honig No rights reserved"
- board text added: "FUNCTION"
- board text added: "SELECT"
- board text removed: "(c) deFEEST WTF"
- board text removed: "C64 Shield V0.42"
- board text removed: "DOWN"
- board text removed: "Get Started at CompShield.GadgetFactory.Net"
- board text removed: "LEFT"
- board text removed: "PS/2 A"
- board text removed: "RIGHT"
- board text removed: "UP"

Commit message: Moved some vias around to balance the return currents more.
Parts:
- moved R17 11.9 mm to (139.7, 109.2), turned to 0 degrees
- moved S1 4.45 mm to (165.1, 116.8)
- moved S3 4.45 mm to (137.8, 116.8)
- moved R9 3.42 mm to (160.0, 110.5)
- moved R10 1.27 mm to (146.1, 109.2), turned to 0 degrees
- moved S2 0.64 mm to (151.1, 113.0)
Connections:
- AJ2 pad LS: (no net) -> Net-(AJ2-PadLS)
- AJ2 pad RS: (no net) -> Net-(AJ2-PadRS)
- H1 pad D13: (no net) -> Net-(H1-PadD13)
- H1 pad D20: (no net) -> SW_SELECT
- H1 pad D21: (no net) -> SW_RESET
- H1 pad D28: SW_SELECT -> D28
- H1 pad D30: SW_RESET -> D30
- H1 pad RES: (no net) -> Net-(H1-PadRES)
- H1 pad RX: (no net) -> /BPS6001 Classic Computing Shield_1/RX
- H1 pad TX: (no net) -> /BPS6001 Classic Computing Shield_1/TX
- H1 pad VIN: (no net) -> Net-(H1-PadVIN)
- PS2_B1 pad 2: (no net) -> Net-(PS2_B1-Pad2)
- PS2_B1 pad 6: (no net) -> Net-(PS2_B1-Pad6)
- PWR_1 pad P2: (no net) -> Net-(PWR_1-PadP2)
- PWR_1 pad P4: (no net) -> Net-(PWR_1-PadP4)
- PWR_2 pad P2: (no net) -> Net-(PWR_2-PadP2)
- SD1 pad 1: (no net) -> Net-(SD1-Pad1)
- SD1 pad 8: (no net) -> Net-(SD1-Pad8)
- SD1 pad CD1: (no net) -> SD_CD
- SD1 pad CD2: (no net) -> Net-(SD1-PadCD2)
- X1 pad 12: (no net) -> Net-(X1-Pad12)
- X1 pad 15: (no net) -> Net-(X1-Pad15)
- X1 pad 4: (no net) -> Net-(X1-Pad4)
- X1 pad 5: (no net) -> Net-(X1-Pad5)
- X1 pad 9: (no net) -> Net-(X1-Pad9)
Routing:
- net 3V3_PWR6: track 219.9 -> 237.8 mm
- net SW_SELECT: track 52.3 -> 44.9 mm, vias 1 -> 0
- net GREEN4: track 21.6 -> 27.6 mm
- net SD_MISO: track 56.8 -> 62.4 mm
- net BLUE2: track 36.9 -> 42.5 mm
- net SW_FUNCTION: track 20.9 -> 25.3 mm
- net SD_MOSI: track 62.3 -> 66.4 mm
- net SD_~CS: track 71.0 -> 67.6 mm
- net SD_SCK: track 64.5 -> 66.6 mm
- net SW_RESET: track 35.6 -> 37.7 mm, vias 1 -> 0
- net BLUE1: track 43.7 -> 42.1 mm
- net VERTICAL_SYNC: track 47.3 -> 45.7 mm
- net HORIZONTAL_SYNC: track 50.7 -> 49.4 mm
- net GREEN3: track 23.7 -> 22.5 mm
- net JS1_5: track 66.2 -> 67.3 mm
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